File: tps/tp2/pcb/kicad/flyback_pcb.kicad_sch (KiCad schematic)
At the start: 49 parts, among them J1 Bornera, J2 Conn_01x11_Pin, J3 Conn_01x11_Pin, J4 Bornera, J5 Bornera, J6 Bornera, Q1 BUZ80, U1 UC3526N

Commit message: fix transformer pin assignments
Connections:
- net DRAIN: now also J2.3 (Pin_3); no longer J2.5 (Pin_5)
- net GND1: now also J3.9 (Pin_9); no longer J3.11 (Pin_11)
- net GND2: now also J3.4 (Pin_4); no longer J3.2 (Pin_2)
- net VL1: now also J2.2 (Pin_2); no longer J2.7 (Pin_7)
- net VL16V: now also J3.8 (Pin_8); no longer J3.10 (Pin_10)
- net VL5V: now also J3.2 (Pin_2); no longer J3.1 (Pin_1)
Other:
- note added: "Puntito"
Changed lines of the file:
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@@
+		)
+	)
+	(text "Puntito"
+		(exclude_from_sim no)
+		(at 229.87 43.688 0)
+		(effects
+			(font
+				(size 1.27 1.27)
+				(italic yes)
+			)
 		)
 	)
@@
 		(exclude_from_sim no)
 		(at 68.58 137.668 0)
+		(effects
+			(font
+				(size 1.27 1.27)
+				(italic yes)
+			)
+		)
+	)
+	(text "Puntito"
+		(exclude_from_sim no)
+		(at 192.278 45.974 0)
+		(effects
+			(font
+				(size 1.27 1.27)
+				(italic yes)
+			)
+		)
+	)
+	(text "Puntito"
+		(exclude_from_sim no)
+		(at 228.6 28.448 0)
 		(effects
 			(font
@@
 	(wire
 		(pts
+			(xy 39.37 67.31) (xy 55.88 67.31)
+		)
+		(stroke
+			(width 0)
+			(type default)
+		)
+	)
+	(wire
+		(pts
+			(xy 73.66 139.7) (xy 83.82 139.7)
+		)
+		(stroke
+			(width 0)
+			(type default)
+		)
+	)
+	(wire
+		(pts
+			(xy 85.09 34.29) (xy 105.41 34.29)
+		)
+		(stroke
+			(width 0)
+			(type default)
+		)
+	)
+	(wire
+		(pts
 			(xy 226.06 24.13) (xy 231.14 24.13)
 		)
@@
 	(wire
 		(pts
-			(xy 39.37 67.31) (xy 55.88 67.31)
-		)
-		(stroke
-			(width 0)
-			(type default)
-		)
-	)
-	(wire
-		(pts
-			(xy 73.66 139.7) (xy 83.82 139.7)
-		)
-		(stroke
-			(width 0)
-			(type default)
-		)
-	)
-	(wire
-		(pts
-			(xy 85.09 34.29) (xy 105.41 34.29)
-		)
-		(stroke
-			(width 0)
-			(type default)
-		)
-	)
-	(wire
-		(pts
 			(xy 146.05 120.65) (xy 158.75 120.65)
 		)
@@
 	(wire
 		(pts
-			(xy 226.06 44.45) (xy 231.14 44.45)
-		)
-		(stroke
-			(width 0)
-			(type default)
-		)
-	)
-	(wire
-		(pts
 			(xy 181.61 60.96) (xy 185.42 60.96)
 		)
@@
 	(wire
 		(pts
+			(xy 226.06 29.21) (xy 231.14 29.21)
+		)
+		(stroke
+			(width 0)
+			(type default)
+		)
+	)
+	(wire
+		(pts
 			(xy 31.75 161.29) (xy 50.8 161.29)
 		)
@@
 	(wire
 		(pts
+			(xy 226.06 41.91) (xy 231.14 41.91)
+		)
+		(stroke
+			(width 0)
+			(type default)
+		)
+	)
+	(wire
+		(pts
 			(xy 38.1 88.9) (xy 53.34 88.9)
 		)
@@
 	(wire
 		(pts
-			(xy 191.77 36.83) (xy 198.12 36.83)
-		)
-		(stroke
-			(width 0)
-			(type default)
-		)
-	)
-	(wire
-		(pts
 			(xy 262.89 90.17) (xy 270.51 90.17)
 		)
@@
 	(wire
 		(pts
+			(xy 191.77 41.91) (xy 198.12 41.91)
+		)
+		(stroke
+			(width 0)
+			(type default)
+		)
+	)
+	(wire
+		(pts
 			(xy 160.02 92.71) (xy 176.53 92.71)
 		)
@@
 	(wire
 		(pts
-			(xy 231.14 46.99) (xy 231.14 48.26)
-		)
-		(stroke
-			(width 0)
-			(type default)
-		)
-	)
-	(wire
-		(pts
 			(xy 105.41 34.29) (xy 107.95 34.29)
 		)
@@
 	(wire
 		(pts
-			(xy 226.06 21.59) (xy 231.14 21.59)
-		)
-		(stroke
-			(width 0)
-			(type default)
-		)
-	)
-	(wire
-		(pts
 			(xy 250.19 24.13) (xy 256.54 24.13)
 		)
@@
 	(wire
 		(pts
+			(xy 226.06 39.37) (xy 231.14 39.37)
+		)
+		(stroke
+			(width 0)
+			(type default)
+		)
+	)
+	(wire
+		(pts
 			(xy 250.19 31.75) (xy 256.54 31.75)
 		)
@@
 	(wire
 		(pts
-			(xy 226.06 46.99) (xy 231.14 46.99)
-		)
-		(stroke
-			(width 0)
-			(type default)
-		)
-	)
-	(wire
-		(pts
 			(xy 87.63 139.7) (xy 83.82 139.7)
 		)
@@
 	(wire
 		(pts
-			(xy 231.14 24.13) (xy 231.14 25.4)
-		)
-		(stroke
-			(width 0)
-			(type default)
-		)
-	)
-	(wire
-		(pts
 			(xy 278.13 90.17) (xy 278.13 92.71)
 		)
@@
 	(wire
 		(pts
+			(xy 191.77 44.45) (xy 198.12 44.45)
+		)
+		(stroke
+			(width 0)
+			(type default)
+		)
+	)
+	(wire
+		(pts
 			(xy 46.99 171.45) (xy 46.99 175.26)
 		)
@@
 		(pts
 			(xy 146.05 125.73) (xy 158.75 125.73)
-		)
-		(stroke
-			(width 0)
-			(type default)
-		)
-	)
-	(wire
-		(pts
-			(xy 191.77 31.75) (xy 198.12 31.75)
 		)
 		(stroke
@@
 	)
 	(label "VL1"
+		(at 191.77 44.45 180)
+		(effects
+			(font
+				(size 1.27 1.27)
+			)
+			(justify right bottom)
+		)
+	)
+	(label "VL1"
 		(at 271.78 22.86 0)
 		(effects
@@
 		)
 	)
-	(label "VL16V"
-		(at 231.14 44.45 0)
+	(label "VL5V"
+		(at 231.14 24.13 0)
 		(effects
 			(font
@@
 	)
 	(label "DRAIN"
-		(at 191.77 36.83 180)
-		(effects
-			(font
-				(size 1.27 1.27)
-			)
-			(justify right bottom)
-		)
-	)
-	(label "DRAIN"
 		(at 271.78 52.07 0)
 		(effects
@@
 			)
 			(justify left bottom)
-		)
-	)
-	(label "VL1"
-		(at 191.77 31.75 180)
-		(effects
-			(font
-				(size 1.27 1.27)
-			)
-			(justify right bottom)
 		)
 	)
@@
 		)
 	)
+	(label "DRAIN"
+		(at 191.77 41.91 180)
+		(effects
+			(font
+				(size 1.27 1.27)
+			)
+			(justify right bottom)
+		)
+	)
 	(label "VL1"
 		(at 68.58 30.48 0)
@@
 		)
 	)
+	(label "VL16V"
+		(at 231.14 39.37 0)
+		(effects
+			(font
+				(size 1.27 1.27)
+			)
+			(justify left bottom)
+		)
+	)
 	(label "VL1"
 		(at 248.92 76.2 180)
@@
 			)
 			(justify right bottom)
-		)
-	)
-	(label "VL5V"
-		(at 231.14 21.59 0)
-		(effects
-			(font
-				(size 1.27 1.27)
-			)
-			(justify left bottom)
 		)
 	)
@@
 	(symbol
 		(lib_id "power:GND2")
-		(at 231.14 25.4 0)
+		(at 231.14 29.21 90)
 		(unit 1)
 		(exclude_from_sim no)
@@
 		(fields_autoplaced yes)
 		(property "Reference" "#PWR02"
-			(at 231.14 31.75 0)
+			(at 237.49 29.21 0)
 			(effects
 				(font
@@
 		)
 		(property "Value" "GND2"
-			(at 231.14 30.48 0)
-			(effects
-				(font
-					(size 1.27 1.27)
-				)
+			(at 234.95 29.2099 90)
+			(effects
+				(font
+					(size 1.27 1.27)
+				)
+				(justify right)
 			)
 		)
 		(property "Footprint" ""
-			(at 231.14 25.4 0)
+			(at 231.14 29.21 0)
 			(effects
 				(font
@@
 		)
 		(property "Datasheet" ""
-			(at 231.14 25.4 0)
+			(at 231.14 29.21 0)
 			(effects
 				(font
@@
 		)
 		(property "Description" "Power symbol creates a global label with name \"GND2\" , ground"
-			(at 231.14 25.4 0)
+			(at 231.14 29.21 0)
 			(effects
 				(font
@@
 		)
 		(instances
-			(project ""
+			(project "flyback_pcb"
 				(path "/847a25f2-0901-4b4c-9f93-5b1d0db6f010"
 					(reference "#PWR02")
@@
 	(symbol
 		(lib_id "power:GND1")
-		(at 231.14 48.26 0)
+		(at 231.14 41.91 90)
 		(unit 1)
 		(exclude_from_sim no)
@@
 		(fields_autoplaced yes)
 		(property "Reference" "#PWR010"
-			(at 231.14 54.61 0)
+			(at 237.49 41.91 0)
 			(effects
 				(font
@@
 		)
 		(property "Value" "GND1"
-			(at 231.14 53.34 0)
-			(effects
-				(font
-					(size 1.27 1.27)
-				)
+			(at 234.95 41.9099 90)
+			(effects
+				(font
+					(size 1.27 1.27)
+				)
+				(justify right)
 			)
 		)
 		(property "Footprint" ""
-			(at 231.14 48.26 0)
+			(at 231.14 41.91 0)
 			(effects
 				(font
@@
 		)
 		(property "Datasheet" ""
-			(at 231.14 48.26 0)
+			(at 231.14 41.91 0)
 			(effects
 				(font
@@
 		)
 		(property "Description" "Power symbol creates a global label with name \"GND1\" , ground"
-			(at 231.14 48.26 0)
-			(effects
-				(font
+			(at 231.14 41.91 0)
+			(effects
+				(font

Commit message: routeado sin circuito de switching (UC3526)
Parts:
- added JP5: open, Jumper:SolderJumper-2_P1.3mm_Open_Pad1.0x1.5mm, symbol Jumper:SolderJumper_2_Open
- R1, R10, R11, R12, R3, R4, R6, R8, R9, RD1, RT1: footprint Resistor_THT:R_Axial_DIN0411_L9.9mm_D3.6mm_P12.70mm_Horizontal -> Resistor_THT:R_Axial_DIN0207_L6.3mm_D2.5mm_P7.62mm_Horizontal
Connections:
- net DRAIN: now also J2.9 (Pin_9); no longer J2.3 (Pin_3)
- net GND1: now also J3.3 (Pin_3), JP5.1 (A); no longer J3.9 (Pin_9)
- net GND2: now also J3.8 (Pin_8); no longer J3.4 (Pin_4)
- net VL1: now also J2.10 (Pin_10); no longer J2.2 (Pin_2)
- net VL16V: now also J3.4 (Pin_4); no longer J3.8 (Pin_8)
- net VL5V: now also J3.10 (Pin_10); no longer J3.2 (Pin_2)
- net at RD1.2, U1.11 (RD): now also JP5.2 (B)

Commit message: 1era versión pcb a fabricar
Parts:
- removed C8: 100n-25V, Capacitor_THT:C_Disc_D4.3mm_W1.9mm_P5.00mm, symbol Device:C
- removed D8: 1N4001, Diode_THT:D_DO-41_SOD81_P10.16mm_Horizontal, symbol Diode:1N4001
- added J7: Conn_01x02_Pin, Connector_PinHeader_2.54mm:PinHeader_1x02_P2.54mm_Vertical, symbol Connector:Conn_01x02_Pin
- added TP1, TP2, TP3, TP4, TP5, TP6, TP7, TP8: TestPoint, Connector_Pin:Pin_D1.0mm_L10.0mm, symbol Connector:TestPoint
- C2: value 100u-600V -> 100u-450V; footprint Capacitor_THT:CP_Radial_D14.0mm_P5.00mm -> Capacitor_THT:CP_Radial_D17.0mm_P7.50mm
- C3: value 1u-600V -> 1u-650V; footprint Capacitor_THT:C_Disc_D4.3mm_W1.9mm_P5.00mm -> Capacitor_THT:C_Rect_L27.0mm_W9.0mm_P22.00mm
- C6: footprint Capacitor_THT:CP_Radial_D14.0mm_P5.00mm -> Capacitor_THT:CP_Radial_D7.5mm_P2.50mm
- D3: value 1N4006 -> 1N4008
- R2: footprint Resistor_SMD:R_0805_2012Metric_Pad1.20x1.40mm_HandSolder -> Resistor_THT:R_Axial_DIN0207_L6.3mm_D2.5mm_P7.62mm_Horizontal
Connections:
- net COMP: now also TP8.1
- net CONTROL: now also TP4.1
- net DRAIN: now also TP5.1
- net ERROR+: now also TP7.1
- net ERROR-: now also TP6.1
- net GND1: now also R2.2, U1.6 (-CURRENT_SENSE), U1.7 (+CURRENT_SENSE), J7.1 (Pin_1), J7.2 (Pin_2)
- net GND2: no longer R2.2
- net VL1: now also TP1.1
- net VREF: now also TP2.1
- net at J6.1 (Pin_1): now also JP1.1 (A)
- net GATE: no longer names the net of Q1.1 (G), R4.2
- net GATE: now also TP3.1
- no-connect marks 4 -> 2
Other:
- moved on the sheet: C6, C7
