File: tps/tp2/pcb/kicad/flyback_pcb.kicad_pcb (KiCad board)
At the start: 2 copper layers, 49 parts, among them J1 Bornera, J2 Conn_01x11_Pin, J3 Conn_01x11_Pin, J4 Bornera, J5 Bornera, J6 Bornera, Q1 BUZ80, U1 UC3526N

Commit message: routeado sin circuito de switching (UC3526)
Parts:
- added JP5: open, Jumper:SolderJumper-2_P1.3mm_Open_Pad1.0x1.5mm, B.Cu at (-48.1, 103.6)
- R1, R10, R11, R12, R3, R4, R6, R8, R9, RD1, RT1: footprint Resistor_THT:R_Axial_DIN0411_L9.9mm_D3.6mm_P12.70mm_Horizontal -> Resistor_THT:R_Axial_DIN0207_L6.3mm_D2.5mm_P7.62mm_Horizontal
- R2, R5, R7: moved to B.Cu
- moved J5 307.3 mm to (217.4, 97.0), turned to -90 degrees
- moved J4 306.6 mm to (217.4, 68.1), turned to -90 degrees
- moved D6 289.7 mm to (196.6, 93.0), turned to 90 degrees
- moved D5 287.3 mm to (196.6, 64.0), turned to 90 degrees
- moved R5 283.1 mm to (199.1, 58.9), turned to 180 degrees
- moved R7 279.0 mm to (197.1, 87.9), turned to 180 degrees
- moved C4 275.4 mm to (196.1, 68.1), turned to -90 degrees
- moved C9 275.4 mm to (195.1, 96.6), turned to -90 degrees
- moved C5 255.4 mm to (205.2, 67.8), turned to -90 degrees
- moved C10 254.8 mm to (204.7, 96.8), turned to -90 degrees
- moved J6 250.9 mm to (141.0, -14.2)
- moved JP1 244.8 mm to (135.1, -29.5)
- moved D4 233.4 mm to (205.2, 58.9), turned to -90 degrees
- moved D7 232.4 mm to (204.7, 87.4), turned to -90 degrees
- moved R6 231.8 mm to (143.8, -30.0)
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Connections:
- J2 pad 10: unconnected-(J2-Pin_10-Pad10) -> /VL1
- J2 pad 2: /VL1 -> unconnected-(J2-Pin_2-Pad2)
- J2 pad 3: /DRAIN -> unconnected-(J2-Pin_3-Pad3)
- J2 pad 9: unconnected-(J2-Pin_9-Pad9) -> /DRAIN
- J3 pad 10: unconnected-(J3-Pin_10-Pad10) -> /VL5V
- J3 pad 2: /VL5V -> unconnected-(J3-Pin_2-Pad2)
- J3 pad 3: unconnected-(J3-Pin_3-Pad3) -> GND1
- J3 pad 4: GND2 -> /VL16V
- J3 pad 8: /VL16V -> GND2
- J3 pad 9: GND1 -> unconnected-(J3-Pin_9-Pad9)
Routing:
- net GND1: track 0.00 -> 74.0 mm
- net /VL1: track 0.00 -> 65.0 mm
- net GND2: track 0.00 -> 53.7 mm
- net +16V: track 0.00 -> 33.6 mm
- net +5V: track 0.00 -> 32.2 mm
- net /DRAIN: track 0.00 -> 19.4 mm
- net /VL16V: track 0.00 -> 19.4 mm
- net /VL5V: track 0.00 -> 18.9 mm
- net NEUT: track 0.00 -> 10.8 mm
- net LINE: track 0.00 -> 10.8 mm
- net Net-(C1-Pad2): track 0.00 -> 9.86 mm
- net Net-(D7-K): track 0.00 -> 6.83 mm
- net Net-(D4-K): track 0.00 -> 5.10 mm
- net Net-(D3-K): track 0.00 -> 4.89 mm

Commit message: 1era versión pcb a fabricar
Parts:
- removed C8: 100n-25V, Capacitor_THT:C_Disc_D4.3mm_W1.9mm_P5.00mm
- removed D8: 1N4001, Diode_THT:D_DO-41_SOD81_P10.16mm_Horizontal
- added J7: Conn_01x02_Pin, Connector_PinHeader_2.54mm:PinHeader_1x02_P2.54mm_Vertical, F.Cu at (111.3, 98.9)
- added TP1: TestPoint, Connector_Pin:Pin_D1.0mm_L10.0mm, F.Cu at (155.2, 124.3)
- added TP2: TestPoint, Connector_Pin:Pin_D1.0mm_L10.0mm, F.Cu at (123.2, 63.6)
- added TP3: TestPoint, Connector_Pin:Pin_D1.0mm_L10.0mm, F.Cu at (128.3, 87.5)
- added TP4: TestPoint, Connector_Pin:Pin_D1.0mm_L10.0mm, F.Cu at (122.6, 79.4)
- added TP5: TestPoint, Connector_Pin:Pin_D1.0mm_L10.0mm, F.Cu at (119.1, 92.1)
- added TP6: TestPoint, Connector_Pin:Pin_D1.0mm_L10.0mm, F.Cu at (106.9, 51.6)
- added TP7: TestPoint, Connector_Pin:Pin_D1.0mm_L10.0mm, F.Cu at (106.9, 46.9)
- C2: value 100u-600V -> 100u-450V; footprint Capacitor_THT:CP_Radial_D14.0mm_P5.00mm -> Capacitor_THT:CP_Radial_D17.0mm_P7.50mm
- C3: value 1u-600V -> 1u-650V; footprint Capacitor_THT:C_Disc_D4.3mm_W1.9mm_P5.00mm -> Capacitor_THT:C_Rect_L27.0mm_W9.0mm_P22.00mm
- C6: footprint Capacitor_THT:CP_Radial_D14.0mm_P5.00mm -> Capacitor_THT:CP_Radial_D7.5mm_P2.50mm
- D3: value 1N4006 -> 1N4008
- R2: footprint Resistor_SMD:R_0805_2012Metric_Pad1.20x1.40mm_HandSolder -> Resistor_THT:R_Axial_DIN0207_L6.3mm_D2.5mm_P7.62mm_Horizontal; moved to F.Cu
- moved C6 231.0 mm to (127.0, 72.6), turned to 90 degrees
- moved RV1 202.0 mm to (111.9, 51.4), turned to 180 degrees
- moved C7 200.9 mm to (121.4, 74.4), turned to 90 degrees
- moved R4 200.0 mm to (128.1, 77.0), turned to -90 degrees
- moved RD1 194.8 mm to (124.3, 89.9), turned to 90 degrees
- moved R2 193.7 mm to (110.6, 114.3), turned to 90 degrees
- moved RV2 193.5 mm to (103.8, 60.2), turned to -90 degrees
- moved R9 188.9 mm to (118.2, 59.8), turned to 180 degrees
- moved R8 188.8 mm to (118.2, 56.4), turned to 180 degrees
- moved R11 183.9 mm to (110.5, 46.4)
- moved JP2 183.7 mm to (103.3, 63.8), turned to -90 degrees
- moved C13 182.1 mm to (102.8, 80.0)
- moved C12 178.4 mm to (98.9, 71.3), turned to 90 degrees
- moved R10 177.2 mm to (106.7, 67.6), turned to -90 degrees
- moved RT1 173.8 mm to (103.3, 89.3)
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Connections:
- net /GATE renamed Net-(Q1-G)
- J6 pad 1: Net-(D8-A) -> Net-(J6-Pin_1)
- JP1 pad 1: Net-(D8-K) -> Net-(J6-Pin_1)
- R2 pad 2: GND2 -> GND1
- U1 pad 6: unconnected-(U1--CURRENT_SENSE-Pad6) -> GND1
- U1 pad 7: unconnected-(U1-+CURRENT_SENSE-Pad7) -> GND1
Routing:
- net GND1: track 74.0 -> 416.1 mm
- net +16V: track 33.6 -> 250.8 mm
- net /VL1: track 65.0 -> 105.3 mm
- net /ERROR+: track 0.00 -> 25.9 mm
- net /ERROR-: track 0.00 -> 23.3 mm
- net /nRESET: track 0.00 -> 13.6 mm
- net /CONTROL: track 0.00 -> 12.3 mm
- net /SOFTSTART: track 0.00 -> 11.9 mm
- net /COMP: track 0.00 -> 11.5 mm
- net Net-(J6-Pin_1): track 0.00 -> 10.6 mm
- net Net-(JP1-B): track 0.00 -> 10.2 mm
- net /VREF: track 0.00 -> 9.66 mm
- net Net-(Q1-G): track 0.00 -> 8.25 mm
- net Net-(JP5-B): track 0.00 -> 7.62 mm
- net +5V: track 32.2 -> 39.1 mm
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- added copper zone on B.Cu, net /VL1
- added copper zone on B.Cu, net GND1
Other:
- board outline added: 133.9 x 95.1 mm
- board text added: "EPot - TP2 - Flyback Mayo 2025 - Grupo3"

Commit message: add routing and 3D views; update footprint dimensions for capacitors
Parts:
- added TP8: TestPoint, Connector_Pin:Pin_D1.0mm_L10.0mm, F.Cu at (100.3, 63.0)
- C10, C5: footprint Capacitor_THT:CP_Radial_D14.0mm_P5.00mm -> Capacitor_THT:CP_Radial_D7.5mm_P2.50mm
- moved D4 10.5 mm to (210.3, 80.8)
- moved R5 9.71 mm to (214.9, 80.8)
- moved J4 7.89 mm to (217.2, 75.2)
- moved J5 6.85 mm to (217.2, 100.5)
- moved C5 5.19 mm to (207.8, 73.9)
- moved C10 3.93 mm to (208.0, 99.0)
- moved C4 1.04 mm to (201.7, 74.9)
- moved D5 1.02 mm to (196.1, 75.2)
Routing:
- net +16V: track 250.8 -> 235.8 mm
- net +5V: track 39.1 -> 31.8 mm
- net GND2: track 60.1 -> 53.5 mm
- net GND1: track 416.1 -> 410.9 mm
- net /COMP: track 11.5 -> 16.3 mm
- net /VL5V: track 14.8 -> 13.9 mm
- net Net-(D4-K): track 2.81 -> 3.57 mm
Other:
- board size 133.9 x 95.1 mm -> 126.2 x 95.1 mm
- board text added: "EPot - TP2 Flyback Mayo 2025 Grupo3"
- board text removed: "EPot - TP2 - Flyback Mayo 2025 - Grupo3"
