File: tps/tp3/pcb/kicad/inverter.kicad_pcb (KiCad board)
At the start: 2 copper layers, 100 x 150 mm, 106 parts, among them J1 220Vac In, J2 Motor, J3 5Vext In, J4 Conn_01x03_Pin, J5 Conn_01x03_Pin, J6 15Vext In, J7 Vd out, J8 Conn_01x03_Pin, Q1 IRF820, Q2 IRF820, Q3 IRF820, Q4 IRF820, Q5 IRF820, Q6 IRF820, U1 IR2110-A, U2 IR2110-B, U3 IR2110-C, U4 ESP32-DEVKIT-V1

Commit message: pcb aprobado por Victor y Pablo
Parts:
- moved C22 43.1 mm to (153.8, 80.5)
- moved D7 43.1 mm to (154.5, 69.2)
- moved R15 43.1 mm to (156.5, 73.5)
- moved J6 43.1 mm to (153.7, 74.5)
- moved U4 3.96 mm to (107.3, 50.0)
Routing:
- net /OUT_A: track 64.2 -> 72.3 mm
- net COM: vias 0 -> 4
- added copper zone on B.Cu, net COM
Changed lines of the file:
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@@
 			(psa4output no)
 			(plot_black_and_white yes)
-			(plotinvisibletext no)
 			(sketchpadsonfab no)
 			(plotpadnumbers no)
@@
 	(footprint "Capacitor_THT:C_Disc_D4.7mm_W2.5mm_P5.00mm"
 		(layer "F.Cu")
-		(at 190.5 58 -90)
+		(at 153.75 80.5 -90)
 		(descr "C, Disc series, Radial, pin pitch=5.00mm, diameter*width=4.7*2.5mm^2, Capacitor, http://www.vishay.com/docs/45233/krseries.pdf")
 		(tags "C Disc series Radial pin pitch 5.00mm diameter 4.7mm width 2.5mm Capacitor")
@@
 	(footprint "esp32devkitv1:MODULE_ESP32_DEVKIT_V1"
 		(layer "F.Cu")
-		(at 103.526 48.895 90)
+		(at 107.315 50.05 90)
 		(property "Reference" "U4"
 			(at -11.355 -27.36 90)
@@
 			(polygon
 				(pts
-					(xy 122.511 57.805) (xy 122.511 40.115) (xy 129.001 40.115) (xy 129.001 57.805)
+					(xy 126.3 58.96) (xy 126.3 41.27) (xy 132.79 41.27) (xy 132.79 58.96)
 				)
 			)
@@
 			(polygon
 				(pts
-					(xy 122.511 57.805) (xy 122.511 40.115) (xy 129.001 40.115) (xy 129.001 57.805)
+					(xy 126.3 58.96) (xy 126.3 41.27) (xy 132.79 41.27) (xy 132.79 58.96)
 				)
 			)
@@
 			(polygon
 				(pts
-					(xy 122.511 57.805) (xy 122.511 40.115) (xy 129.001 40.115) (xy 129.001 57.805)
+					(xy 126.3 58.96) (xy 126.3 41.27) (xy 132.79 41.27) (xy 132.79 58.96)
 				)
 			)
@@
 	(footprint "LED_THT:LED_D3.0mm"
 		(layer "F.Cu")
-		(at 191.29 46.75 180)
+		(at 154.54 69.25 180)
 		(descr "LED, diameter 3.0mm, 2 pins, generated by kicad-footprint-generator")
 		(tags "LED")
@@
 		(pad "1" thru_hole circle
 			(at 0 0 135)
-			(size 1.6 1.6)
-			(drill 0.8)
+			(size 2 2)
+			(drill 1)
 			(layers "*.Cu" "*.Mask")
 			(remove_unused_layers no)
@@
 	(footprint "Connector_Molex:Molex_KK-254_AE-6410-02A_1x02_P2.54mm_Vertical"
 		(layer "F.Cu")
-		(at 190.48 51.975 -90)
+		(at 153.73 74.475 -90)
 		(descr "Molex KK-254 Interconnect System, old/engineering part number: AE-6410-02A example for new part number: 22-27-2021, 2 Pins (http://www.molex.com/pdm_docs/sd/022272021_sd.pdf), generated with kicad-footprint-generator")
 		(tags "connector Molex KK-254 vertical")
@@
 	(footprint "Resistor_SMD:R_0805_2012Metric_Pad1.20x1.40mm_HandSolder"
 		(layer "B.Cu")
-		(at 193.25 51 90)
+		(at 156.5 73.5 90)
 		(descr "Resistor SMD 0805 (2012 Metric), square (rectangular) end terminal, IPC-7351 nominal with elongated pad for handsoldering. (Body size source: IPC-SM-782 page 72, https://www.pcb-3d.com/wordpress/wp-content/uploads/ipc-sm-782a_amendment_1_and_2.pdf), generated with kicad-footprint-generator")
 		(tags "resistor handsolder")
@@
 	)
 	(segment
+		(start 83.75 124.533737)
+		(end 81.990935 126.292802)
+		(width 1.5)
+		(layer "B.Cu")
+		(net 2)
+	)
+	(segment
 		(start 78.010364 96.487636)
 		(end 78.010364 98.642898)
@@
 	)
 	(segment
-		(start 89.89356 121.982279)
-		(end 97.344279 121.982279)
-		(width 2)
+		(start 82.5 103.132533)
+		(end 82.5 121.25)
+		(width 1.5)
 		(layer "B.Cu")
 		(net 2)
 	)
 	(segment
-		(start 82.5 103.132533)
-		(end 82.5 119.5)
+		(start 82.5 121.25)
+		(end 83.75 122.5)
 		(width 1.5)
 		(layer "B.Cu")
@@
 	)
 	(segment
+		(start 89.89356 121.982279)
+		(end 97.344279 121.982279)
+		(width 2)
+		(layer "B.Cu")
+		(net 2)
+	)
+	(segment
 		(start 101.092 131.064)
 		(end 101.092 134.62)
@@
 	)
 	(segment
-		(start 98.044 128.016)
-		(end 101.092 131.064)
-		(width 2)
+		(start 83.75 122.5)
+		(end 83.75 124.533737)
+		(width 1.5)
 		(layer "B.Cu")
 		(net 2)
 	)
 	(segment
-		(start 80.524836 101.157369)
-		(end 82.5 103.132533)
-		(width 1.5)
+		(start 98.044 128.016)
+		(end 101.092 131.064)
+		(width 2)
 		(layer "B.Cu")
 		(net 2)
@@
 	)
 	(segment
+		(start 80.524836 101.157369)
+		(end 82.5 103.132533)
+		(width 1.5)
+		(layer "B.Cu")
+		(net 2)
+	)
+	(segment
 		(start 82.704846 91.793154)
 		(end 78.010364 96.487636)
@@
 		(net 2)
 	)
+	(via
+		(at 63.25 150.5)
+		(size 3)
+		(drill 1)
+		(layers "F.Cu" "B.Cu")
+		(free yes)
+		(net 3)
+	)
+	(via
+		(at 99.75 151.25)
+		(size 3)
+		(drill 1)
+		(layers "F.Cu" "B.Cu")
+		(free yes)
+		(net 3)
+	)
+	(via
+		(at 117.75 151.25)
+		(size 3)
+		(drill 1)
+		(layers "F.Cu" "B.Cu")
+		(free yes)
+		(net 3)
+	)
+	(via
+		(at 145.75 151.75)
+		(size 3)
+		(drill 1)
+		(layers "F.Cu" "B.Cu")
+		(free yes)
+		(net 3)
+	)
 	(segment
 		(start 91 90)
@@
 	)
 	(segment
-		(start 192.3575 56.3925)
-		(end 193 57.035)
+		(start 155.6075 78.8925)
+		(end 156.25 79.535)
 		(width 1)
 		(layer "B.Cu")
@@
 	)
 	(segment
-		(start 190.48 54.515)
-		(end 192.3575 56.3925)
+		(start 153.73 77.015)
+		(end 155.6075 78.8925)
 		(width 1)
 		(layer "B.Cu")
@@
 	)
 	(segment
-		(start 193 57.035)
-		(end 193 60.5)
+		(start 156.25 79.535)
+		(end 156.25 83)
 		(width 1)
 		(layer "B.Cu")
@@
 	)
 	(segment
-		(start 193.25 52)
-		(end 193.25 55.5)
+		(start 156.5 74.5)
+		(end 156.5 78)
 		(width 1)
 		(layer "B.Cu")
@@
 	)
 	(segment
-		(start 193.25 55.5)
-		(end 192.3575 56.3925)
+		(start 156.5 78)
+		(end 155.6075 78.8925)
 		(width 1)
 		(layer "B.Cu")
@@
 	)
 	(segment
-		(start 193 60.5)
-		(end 190.5 63)
+		(start 156.25 83)
+		(end 153.75 85.5)
 		(width 1)
 		(layer "B.Cu")
@@
 	)
 	(segment
-		(start 188.75 58)
-		(end 190.5 58)
+		(start 152 80.5)
+		(end 153.75 80.5)
 		(width 1)
 		(layer "B.Cu")
@@
 	)
 	(segment
-		(start 190.48 51.975)
-		(end 189.025 51.975)
+		(start 153.73 74.475)
+		(end 152.275 74.475)
 		(width 1)
 		(layer "B.Cu")
@@
 	)
 	(segment
-		(start 188.75 46.75)
-		(end 188.75 50)
+		(start 152 69.25)
+		(end 152 72.5)
 		(width 1)
 		(layer "B.Cu")
@@
 	)
 	(segment
-		(start 187.25 56.5)
-		(end 188.75 58)
+		(start 150.5 79)
+		(end 152 80.5)
 		(width 1)
 		(layer "B.Cu")
@@
 	)
 	(segment
-		(start 190.48 51.975)
-		(end 188.6275 50.1225)
+		(start 153.73 74.475)
+		(end 151.8775 72.6225)
 		(width 1)
 		(layer "B.Cu")
@@
 	)
 	(segment
-		(start 189.025 51.975)
-		(end 187.25 53.75)
+		(start 152.275 74.475)
+		(end 150.5 76.25)
 		(width 1)
 		(layer "B.Cu")
@@
 	)
 	(segment
-		(start 187.25 53.75)
-		(end 187.25 56.5)
+		(start 150.5 76.25)
+		(end 150.5 79)
 		(width 1)
 		(layer "B.Cu")
@@
 	)
 	(segment
-		(start 193.25 47.75)
-		(end 193.25 50)
+		(start 156.5 70.25)
+		(end 156.5 72.5)
 		(width 1)
 		(layer "B.Cu")
@@
 	)
 	(segment
-		(start 192.25 46.75)
-		(end 193.25 47.75)
+		(start 155.5 69.25)
+		(end 156.5 70.25)
 		(width 1)
 		(layer "B.Cu")
@@
 	)
 	(segment
-		(start 191.29 46.75)
-		(end 192.25 46.75)
+		(start 154.54 69.25)
+		(end 155.5 69.25)
 		(width 1)
 		(layer "B.Cu")
@@
 		(layer "F.Cu")
 		(hatch edge 0.5)
+		(priority 1)
+		(connect_pads
+			(clearance 1.5)
+		)
+		(min_thickness 0.25)
+		(filled_areas_thickness no)
+		(fill yes
+			(thermal_gap 0.5)
+			(thermal_bridge_width 0.5)
+			(smoothing fillet)
+			(radius 2)
+		)
+		(polygon
+			(pts
+				(xy 123.833071 136.874472) (xy 112.833071 126.124472) (xy 126.432833 111.754912) (xy 137.425999 122.997923)
+				(xy 124.333071 137.374472)
+			)
+		)
+	)
+	(zone
+		(net 3)
+		(net_name "COM")
+		(layer "F.Cu")
+		(hatch edge 0.5)
+		(connect_pads
+			(clearance 1.5)
+		)
+		(min_thickness 0.25)
+		(filled_areas_thickness no)
+		(fill yes
+			(thermal_gap 0.5)
+			(thermal_bridge_width 0.5)
+			(smoothing fillet)
+			(radius 2)
+		)
+		(polygon
+			(pts
+				(xy 156.25 155.5) (xy 156 60) (xy 56.5 60) (xy 56.5 156) (xy 156.25 155.75)
+			)
+		)
+	)
+	(zone
+		(net 3)
+		(net_name "COM")
+		(layer "F.Cu")
+		(hatch edge 0.5)
+		(priority 2)
+		(connect_pads
+			(clearance 1.5)
+		)
+		(min_thickness 0.25)
+		(filled_areas_thickness no)
+		(fill yes
+			(thermal_gap 0.5)
+			(thermal_bridge_width 0.5)
+			(smoothing fillet)
+			(radius 2)
+		)
+		(polygon
+			(pts
+				(xy 97.75 110.5) (xy 114.25 110.5) (xy 114 128) (xy 97.75 128)
+			)
+		)
+	)
+	(zone
+		(net 3)
+		(net_name "COM")
+		(layer "F.Cu")
+		(hatch edge 0.5)
+		(priority 1)
 		(connect_pads
 			(clearance 1.5)
 		)
-		(min_thickness 0.5)
+		(min_thickness 0.25)
 		(filled_areas_thickness no)
 		(fill yes
@@
 		(polygon
 			(pts
-				(xy 156.21 155.702) (xy 156.21 121.158) (xy 124.714 89.662) (xy 86.36 89.662) (xy 56.134 119.888)
-				(xy 56.134 155.702)
+				(xy 75 122.75) (xy 85.75 111.75) (xy 100.11956 125.349762) (xy 88.876549 136.342928) (xy 74.5 123.25)
 			)
 		)
@@
 		(layer "B.Cu")
 		(hatch edge 0.5)
-		(priority 1)
+		(priority 3)
+		(connect_pads
+			(clearance 1.5)
+		)
+		(min_thickness 0.25)
+		(filled_areas_thickness no)
+		(fill yes
+			(thermal_gap 0.5)
+			(thermal_bridge_width 0.5)
+		)
+		(polygon
+			(pts
+				(xy 156.25 144.25) (xy 74.75 144.25) (xy 74.75 137) (xy 156.25 137)
+			)
+		)
+	)
+	(zone
+		(net 3)
+		(net_name "COM")
+		(layer "B.Cu")
+		(hatch edge 0.5)
+		(priority 4)
 		(connect_pads
 			(clearance 1.5)
 		)
-		(min_thickness 0.5)
+		(min_thickness 0.25)
 		(filled_areas_thickness no)
 		(fill yes
@@
 		(polygon
 			(pts
-				(xy 156.21 155.702) (xy 156.21 116.586) (xy 56.134 116.586) (xy 56.134 155.702)
+				(xy 156.25 155.75) (xy 156.25 145.25) (xy 56.5 144.75) (xy 56.5 155.5)
 			)
 		)

Commit message: final inverter pcb
Parts:
- removed C20, C28, C29, C30: 10u-25V, Capacitor_THT:CP_Radial_D4.0mm_P1.50mm
- removed C22: 1u-50V, Capacitor_THT:C_Disc_D4.7mm_W2.5mm_P5.00mm
- removed JP1: Jumper_2_Bridged, Jumper:SolderJumper-2_P1.3mm_Open_RoundedPad1.0x1.5mm
- removed TP19, TP20, TP21, TP22, TP23, TP24: TestPoint, Connector_PinHeader_2.54mm:PinHeader_1x01_P2.54mm_Vertical
- R16, R17, R18, R7, R8: moved to B.Cu
- moved R7 195.5 mm to (63.6, 43.8), turned to 180 degrees
- moved D5 191.4 mm to (68.6, 42.8), turned to 90 degrees
- moved J3 188.9 mm to (60.6, 40.3), turned to 90 degrees
- moved TP26 183.0 mm to (60.4, 138.0)
- moved D6 179.9 mm to (78.5, 68.3)
- moved R8 177.5 mm to (78.6, 62.7), turned to 90 degrees
- moved TP25 168.0 mm to (60.5, 121.2)
- moved TP27 165.0 mm to (68.5, 37.4)
- moved C19 152.2 mm to (78.9, 37.9), turned to -90 degrees
- moved TP1 149.1 mm to (59.0, 88.7)
- moved TP12 148.8 mm to (74.8, 120.5)
- moved TP2 146.8 mm to (61.8, 96.7)
- moved TP11 140.6 mm to (82.5, 113.1)
- moved C24 134.3 mm to (85.9, 68.3)
- moved C17 129.9 mm to (74.0, 37.8), turned to -90 degrees
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Connections:
- C1 pad 2: VSS -> COM
- C17 pad 2: VSS -> COM
- C19 pad 2: VSS -> COM
- C2 pad 2: VSS -> COM
- C23 pad 2: VSS -> COM
- C24 pad 2: VSS -> COM
- C3 pad 2: VSS -> COM
- C4 pad 2: VSS -> COM
- C5 pad 2: VSS -> COM
- C6 pad 2: VSS -> COM
- J3 pad 1: VEXT -> COM
- J3 pad 2: VSS -> VEXT
- R7 pad 2: VSS -> COM
- R8 pad 2: VSS -> COM
- RV1 pad 1: VSS -> COM
- U1 pad 13: VSS -> COM
- U2 pad 13: VSS -> COM
- U3 pad 13: VSS -> COM
- U4 pad 2: VSS -> COM
- U4 pad 23: Net-(J8-Pin_3) -> unconnected-(U4-D25-Pad23)
- U4 pad 24: Net-(J8-Pin_2) -> unconnected-(U4-D26-Pad24)
- U4 pad 25: Net-(J8-Pin_1) -> unconnected-(U4-D27-Pad25)
- U4 pad 29: VSS -> COM
Routing:
- net VDD: track 28.8 -> 240.3 mm
- net COM: track 134.2 -> 264.4 mm, vias 4 -> 13
- net VDRV: track 89.4 -> 219.4 mm, vias 0 -> 6
- net VSS: track 52.8 -> 0.00 mm, vias 3 -> 0
- net Net-(U4-D5): track 0.00 -> 46.7 mm
- net Net-(U4-D15): track 0.00 -> 44.4 mm
- net Net-(U4-TX2): track 0.00 -> 41.8 mm
- net Net-(U4-D2): track 0.00 -> 41.5 mm
- net Net-(U4-D34): track 0.00 -> 38.8 mm
- net VEXT: track 0.00 -> 36.8 mm
- net /HIN_A: track 0.00 -> 19.9 mm
- net /LIN_C: track 0.00 -> 15.0 mm
- net /LIN_A: track 0.00 -> 14.7 mm
- net /HIN_C: track 0.00 -> 14.5 mm
- net /HIN_B: track 0.00 -> 14.0 mm
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Other:
- board size 100 x 150 mm -> 100 x 121 mm
- board text added: "22.28 - EPot TP3 - Inverter - G2 Junio 2025"
