File: tps/tp3/pcb/kicad/inverter.kicad_sch (KiCad schematic)
At the start: 106 parts, among them J1 220Vac In, J2 Motor, J3 5Vext In, J4 Conn_01x03_Pin, J5 Conn_01x03_Pin, J6 15Vext In, J7 Vd out, J8 Conn_01x03_Pin, Q1 IRF820, Q2 IRF820, Q3 IRF820, Q4 IRF820, Q5 IRF820, Q6 IRF820, U1 IR2110-A, U2 IR2110-B, U3 IR2110-C, U4 ESP32-DEVKIT-V1

Commit message: final inverter pcb
Parts:
- removed J8: Conn_01x03_Pin, Connector_PinHeader_2.54mm:PinHeader_1x03_P2.54mm_Vertical, symbol Connector:Conn_01x03_Pin
- removed JP1: Jumper_2_Bridged, Jumper:SolderJumper-2_P1.3mm_Open_RoundedPad1.0x1.5mm, symbol Jumper:Jumper_2_Bridged
- removed TP19, TP20, TP21, TP22, TP23, TP24: TestPoint, Connector_PinHeader_2.54mm:PinHeader_1x01_P2.54mm_Vertical, symbol Connector:TestPoint
Connections:
- net COM: now also C1.2, C17.2, C19.2, C2.2, C23.2, C24.2, C3.2, C4.2, C5.2, C6.2, J3.1 (Pin_1), R7.2, R8.2, RV1.1, U1.13 (VSS), U2.13 (VSS), U3.13 (VSS), U4.2 (GND), U4.29 (GND)
- net VEXT: now also J3.2 (Pin_2); no longer J3.1 (Pin_1)
- removed net VSS: C1.2, C17.2, C19.2, C2.2, C23.2, C24.2, C3.2, C4.2, C5.2, C6.2, J3.2 (Pin_2), R7.2, R8.2, RV1.1, U1.13 (VSS), U2.13 (VSS), U3.13 (VSS), U4.2 (GND), U4.29 (GND)
